File: hardware/Clock_rev1.brd (EAGLE design)
At the start: 233.3 x 138.4 mm, 35 parts

Commit message: Add files via upload
Parts:
- moved CURRLIM2 139.7 mm to (41.9, 83.8)
- moved DECOUP3 139.7 mm to (174.0, 87.6)
- moved CURRLIM0 139.7 mm to (193.0, 101.6)
- moved DECOUP1 139.7 mm to (31.8, 83.8)
- moved MINUTES 139.7 mm to (186.7, 64.8), flipped to the bottom
- moved SECONDS_ONES 139.7 mm to (47.0, 64.8), flipped to the bottom
- moved SP0 139.7 mm to (182.9, 95.2)
- moved SP2 139.7 mm to (40.6, 91.4)
- flipped GREEN_GO to the bottom
- flipped RED1 to the bottom
- flipped RED2 to the bottom
- flipped RED3 to the bottom
- flipped RED4 to the bottom
- flipped RED5 to the bottom
- flipped SECONDS_TENS to the bottom
Routing:
- net 5V: track 236.2 -> 0.00 mm
