File: hardware/Clock/Clock_rev1.brd (EAGLE design)
At the start: 233.3 x 138.4 mm, 35 parts

Commit message: Add files via upload
Parts:
- moved INFARED_1 85.1 mm to (6.35, 21.6), turned to 90 degrees
- moved INFARED_2 81.3 mm to (6.35, 39.4), turned to 90 degrees
- moved CURRLIM0 28.4 mm to (180.3, 76.2), turned to 90 degrees
- moved USB_B_IN 14.0 mm to (6.35, 106.7)
- moved BUTTONS_CONNECTOR 12.8 mm to (5.08, 85.1)
- moved R10 12.8 mm to (21.6, 45.7)
- moved R11 12.8 mm to (17.8, 45.7)
- moved R13 12.8 mm to (29.2, 45.7)
- moved R3 12.8 mm to (25.4, 45.7)
- moved PCB1 11.5 mm to (21.6, 62.2)
- moved R12 11.5 mm to (30.5, 77.5)
- moved R2 11.5 mm to (26.7, 77.5)
- moved D1 6.35 mm to (33.0, 41.9), turned to 270 degrees
- moved CURRLIM2 5.24 mm to (47.0, 85.1)
- moved DECOUP1 5.24 mm to (36.8, 85.1)
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Connections:
- new net N$9: PCB1.RESET@2
- net D0: no longer CURRLIM0.2
- net DP0: now also CURRLIM0.2
- net RST: no longer PCB1.RESET@2
Routing:
- net RST: track 37.6 -> 450.2 mm
- net 5V: track 0.00 -> 318.2 mm, vias 0 -> 2
- net N$8: track 0.00 -> 265.7 mm
- net SS: track 0.00 -> 258.5 mm, vias 0 -> 2
- net N$12: track 0.00 -> 239.4 mm
- net N$16: track 0.00 -> 219.2 mm
- net N$13: track 0.00 -> 205.3 mm
- net N$11: track 0.00 -> 187.9 mm
- net N$1: track 0.00 -> 184.3 mm
- net N$14: track 0.00 -> 173.0 mm
- net 12V: track 0.00 -> 148.2 mm
- net N$15: track 0.00 -> 140.2 mm
- net E2: track 0.00 -> 98.9 mm
- net D2: track 0.00 -> 94.0 mm
- net E0: track 0.00 -> 92.8 mm
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- added copper zone on layer 1, net GND
- added copper zone on layer 16, net GND
