File: hardware/Clock/Clock_rev1.sch (EAGLE design)
At the start: 31 parts

Commit message: Add files via upload
Connections:
- new net N$9: PCB1.RESET@2
- net D0: no longer CURRLIM0.2
- net DP0: now also CURRLIM0.2
- net RST: no longer PCB1.RESET@2
Changed lines of the file:
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@@
-</segment>
-</net>
-<net name="N$7" class="0">
-<segment>
-<pinref part="SP1" gate="G$1" pin="SOUT"/>
-<pinref part="SP2" gate="G$1" pin="SIN"/>
-<wire x1="177.8" y1="223.52" x2="193.04" y2="223.52" width="0.1524" layer="91"/>
 </segment>
 </net>
@@
 <pinref part="PCB1" gate="PCB" pin="RESET"/>
 <wire x1="30.48" y1="236.22" x2="27.94" y2="236.22" width="0.1524" layer="91"/>
-<pinref part="PCB1" gate="PCB" pin="RESET@2"/>
-<wire x1="27.94" y1="233.68" x2="30.48" y2="233.68" width="0.1524" layer="91"/>
-<wire x1="27.94" y1="233.68" x2="27.94" y2="236.22" width="0.1524" layer="91"/>
 <label x="27.94" y="236.22" size="1.778" layer="95"/>
 </segment>
@@
 <label x="91.44" y="220.98" size="1.778" layer="95"/>
 </segment>
+<segment>
+<pinref part="CURRLIM0" gate="G$1" pin="2"/>
+<wire x1="68.58" y1="50.8" x2="71.12" y2="50.8" width="0.1524" layer="91"/>
+<label x="68.58" y="50.8" size="1.778" layer="95"/>
+</segment>
 </net>
 <net name="A0" class="0">
@@
 <wire x1="48.26" y1="53.34" x2="48.26" y2="55.88" width="0.1524" layer="91"/>
 <label x="45.72" y="53.34" size="1.778" layer="95"/>
-</segment>
-<segment>
-<pinref part="CURRLIM0" gate="G$1" pin="2"/>
-<wire x1="68.58" y1="50.8" x2="71.12" y2="50.8" width="0.1524" layer="91"/>
-<label x="68.58" y="50.8" size="1.778" layer="95"/>
 </segment>
 </net>
@@
 </segment>
 </net>
+<net name="N$7" class="0">
+<segment>
+<pinref part="SP1" gate="G$1" pin="SOUT"/>
+<pinref part="SP2" gate="G$1" pin="SIN"/>
+<wire x1="177.8" y1="223.52" x2="193.04" y2="223.52" width="0.1524" layer="91"/>
+</segment>
+</net>
+<net name="N$9" class="0">
+<segment>
+<pinref part="PCB1" gate="PCB" pin="RESET@2"/>
+<wire x1="27.94" y1="233.68" x2="30.48" y2="233.68" width="0.1524" layer="91"/>
+</segment>
+</net>
